File: ErgoDOX pcb/ErgoDOX.kicad_pcb (KiCad board)
At the start: 2 copper layers, 182.8 x 158.9 mm, 66 parts, among them J1 AudioJack4, J5 USB_B_Micro, SW0:10 SW0:3, SW0:11 SW0:2, SW0:12 SW0:1, SW0:7 SW0:6, SW0:8 SW0:5, SW0:9 SW0:4, SW1:10 SW1:3, SW1:11 SW1:2, SW1:12 SW1:1, SW1:13 SW1:0, SW1:9 SW1:4, SW2:10 SW2:3, SW2:11 SW2:2, SW2:12 SW2:1, SW2:13 SW2:0, SW2:7 SW2:6, SW2:8 SW2:5, SW2:9 SW2:4, SW3:10 SW3:3, SW3:11 SW3:2, SW3:12 SW3:1, SW3:13 SW3:0, SW3:8 SW3:5, SW3:9 SW3:4, SW4:10 SW4:3, SW4:11 SW4:2, SW4:12 SW4:1, SW4:13 SW4:0, SW4:7 SW4:6, SW4:8 SW4:5, SW4:9 SW4:4, SW5:10 SW5:3, SW5:11 SW5:2, SW5:12 SW5:1, SW5:13 SW5:0, SW5:7 SW5:6, SW5:8 SW5:5, SW5:9 SW5:4, U1 AT90USB1286-MU, U2 MCP23018, Y1 16MHz

Commit message: Placed diodes, started routing
Parts:
- removed C1, C2: 10p, Capacitors_SMD:C_0603
- removed C3, C4: 1u, Capacitors_SMD:C_0603
- removed C5, C6: 100n, Capacitors_SMD:C_0603
- removed J5: USB_B_Micro, Connectors:USB_Micro-B
- removed R5: 1k, Resistors_SMD:R_0603
- removed SX0:10: SX0:3, ErgoDOX pcb:MX_FLIP_DIODE
- removed SX0:11: SX0:2, ErgoDOX pcb:MX_FLIP_DIODE
- removed Y1: 16MHz, Crystals:Crystal_SMD_2012-2pin_2.0x1.2mm
- added D0:10: D, Diodes_SMD:D_SOD-123, F.Cu at (93.3, 153.5)
- added D0:11: D, Diodes_SMD:D_SOD-123, F.Cu at (66.3, 160.0)
- added D0:12: D, Diodes_SMD:D_SOD-123, F.Cu at (46.3, 172.5)
- added D0:7: D, Diodes_SMD:D_SOD-123, F.Cu at (38.3, 151.5)
- added D0:8: D, Diodes_SMD:D_SOD-123, F.Cu at (60.6, 128.5)
- added D0:9: D, Diodes_SMD:D_SOD-123, F.Cu at (47.3, 167.5)
- added D1:10: D, Diodes_SMD:D_SOD-123, F.Cu at (124.3, 129.5)
- added D1:11: D, Diodes_SMD:D_SOD-123, F.Cu at (143.3, 130.5)
- added D1:12: D, Diodes_SMD:D_SOD-123, F.Cu at (177.3, 139.5)
- added D1:13: D, Diodes_SMD:D_SOD-123, F.Cu at (181.3, 133.5)
- added D1:9: D, Diodes_SMD:D_SOD-123, F.Cu at (105.3, 131.5)
- added D2:10: D, Diodes_SMD:D_SOD-123, F.Cu at (124.3, 110.5)
- added D2:11: D, Diodes_SMD:D_SOD-123, F.Cu at (143.3, 111.5)
- added D2:12: D, Diodes_SMD:D_SOD-123, F.Cu at (251.3, 133.5)
- added D2:13: D, Diodes_SMD:D_SOD-123, F.Cu at (252.3, 96.5)
- added D2:7: D, Diodes_SMD:D_SOD-123, F.Cu at (66.3, 120.0)
- added D2:8: D, Diodes_SMD:D_SOD-123, F.Cu at (85.3, 112.5)
- added D2:9: D, Diodes_SMD:D_SOD-123, F.Cu at (105.3, 111.5)
- added D3:10: D, Diodes_SMD:D_SOD-123, F.Cu at (124.3, 91.5)
- added D3:11: D, Diodes_SMD:D_SOD-123, F.Cu at (143.3, 93.5)
- added D3:12: D, Diodes_SMD:D_SOD-123, F.Cu at (174.3, 114.5)
- added D3:13: D, Diodes_SMD:D_SOD-123, F.Cu at (185.6, 96.5)
- added D3:8: D, Diodes_SMD:D_SOD-123, F.Cu at (86.3, 93.5)
- added D3:9: D, Diodes_SMD:D_SOD-123, F.Cu at (105.3, 92.5)
- added D4:10: D, Diodes_SMD:D_SOD-123, F.Cu at (123.6, 72.5)
- added D4:11: D, Diodes_SMD:D_SOD-123, F.Cu at (143.3, 73.5)
- added D4:12: D, Diodes_SMD:D_SOD-123, F.Cu at (174.3, 94.5)
- added D4:13: D, Diodes_SMD:D_SOD-123, F.Cu at (188.8, 77.5)
- added D4:7: D, Diodes_SMD:D_SOD-123, F.Cu at (68.3, 98.5)
- added D4:8: D, Diodes_SMD:D_SOD-123, F.Cu at (86.3, 74.5)
- added D4:9: D, Diodes_SMD:D_SOD-123, F.Cu at (105.3, 73.5)
- added D5:10: D, Diodes_SMD:D_SOD-123, F.Cu at (124.3, 53.5)
- added D5:11: D, Diodes_SMD:D_SOD-123, F.Cu at (143.3, 54.5)
- added D5:12: D, Diodes_SMD:D_SOD-123, F.Cu at (174.3, 75.5)
- added D5:13: D, Diodes_SMD:D_SOD-123, F.Cu at (189.6, 60.0)
- added D5:7: D, Diodes_SMD:D_SOD-123, F.Cu at (67.3, 56.5)
- added D5:8: D, Diodes_SMD:D_SOD-123, F.Cu at (90.4, 57.5)
- added D5:9: D, Diodes_SMD:D_SOD-123, F.Cu at (105.3, 55.0)
- added J2: USB_B_Micro, Connectors_USB:USB_Micro-B_Wuerth-629105150521, F.Cu at (239.9, 126.2)
- added R10: 0, Resistors_SMD:R_0603, F.Cu at (275.0, 127.5)
- added R9: 0, Resistors_SMD:R_0603, F.Cu at (279.2, 123.6)
- added SW1: TS-1187A-B-A-B, Buttons_Switches_THT:SW_PUSH_6mm, F.Cu at (236.4, 133.6)
- D1:7, D1:8: footprint Diodes_SMD:D_0603 -> Diodes_SMD:D_SOD-123
- J1: footprint ErgoDOX pcb:ASJ-112-M -> ErgoDOX:54-00174
- SW0:10, SW0:11, SW0:12, SW0:7, SW0:8, SW0:9, SW1:10, SW1:11, SW1:12, SW1:13, SW1:9, SW2:10, SW2:11, SW2:12, SW2:13, SW2:7, SW2:8, SW2:9, SW3:10, SW3:11, SW3:12, SW3:13, SW3:8, SW3:9, SW4:10, SW4:11, SW4:12, SW4:13, SW4:7, SW4:8, SW4:9, SW5:10, SW5:11, SW5:12, SW5:13, SW5:7, SW5:8, SW5:9, SX1:7, SX1:8: footprint ErgoDOX pcb:MX_FLIP_DIODE -> ErgoDOX:MX_TOP
- U1: value AT90USB1286-MU -> ATmega32U4-MU; footprint Housings_DFN_QFN:QFN-64-1EP_9x9mm_Pitch0.5mm -> Housings_DFN_QFN:QFN-44-1EP_7x7mm_Pitch0.5mm
- moved U1 111.4 mm to (256.6, 122.1), turned to 0 degrees
- moved SW0:10 9.32 mm to (85.3, 161.5), turned to 25 degrees
- moved SW0:11 8.98 mm to (67.3, 169.5), turned to 25 degrees
- moved D1:7 7.62 mm to (56.3, 142.5), turned to 205 degrees
- moved D1:8 0.28 mm to (73.8, 137.5), turned to 205 degrees
- moved J1 0.24 mm to (91.8, 32.5), turned to 270 degrees
Connections:
- J1 pad R1: /SCLM -> /SCL
- J1 pad R2: /SDAM -> /SDA
- LED_C1 pad 2: Net-(LED_C1-Pad2) -> (no net)
- R1 pad 2: /d+ -> /USB+
- R2 pad 2: /d- -> /USB-
- R6 pad 1: /SDAM -> /SDA
- R7 pad 2: /SCLM -> /SCL
- SW0:12 pad 2: Net-(SW0:12-Pad2) -> Net-(D0:12-Pad2)
- SW0:7 pad 2: Net-(SW0:7-Pad2) -> Net-(D0:7-Pad2)
- SW0:8 pad 2: Net-(SW0:8-Pad2) -> Net-(D0:8-Pad2)
- SW0:9 pad 2: Net-(SW0:9-Pad2) -> Net-(D0:9-Pad2)
- SW1:10 pad 2: Net-(SW1:10-Pad2) -> Net-(D1:10-Pad2)
- SW1:11 pad 2: Net-(SW1:11-Pad2) -> Net-(D1:11-Pad2)
- SW1:12 pad 2: Net-(SW1:12-Pad2) -> Net-(D1:12-Pad2)
- SW1:13 pad 2: Net-(SW1:13-Pad2) -> Net-(D1:13-Pad2)
- SW1:9 pad 2: Net-(SW1:9-Pad2) -> Net-(D1:9-Pad2)
- SW2:10 pad 2: Net-(SW2:10-Pad2) -> Net-(D2:10-Pad2)
- SW2:11 pad 2: Net-(SW2:11-Pad2) -> Net-(D2:11-Pad2)
- SW2:12 pad 2: Net-(SW2:12-Pad2) -> Net-(D2:12-Pad2)
- SW2:13 pad 2: Net-(SW2:13-Pad2) -> Net-(D2:13-Pad2)
- SW2:7 pad 2: Net-(SW2:7-Pad2) -> Net-(D2:7-Pad2)
- SW2:8 pad 2: Net-(SW2:8-Pad2) -> Net-(D2:8-Pad2)
- SW2:9 pad 2: Net-(SW2:9-Pad2) -> Net-(D2:9-Pad2)
- SW3:10 pad 2: Net-(SW3:10-Pad2) -> Net-(D3:10-Pad2)
- SW3:11 pad 2: Net-(SW3:11-Pad2) -> Net-(D3:11-Pad2)
- SW3:12 pad 2: Net-(SW3:12-Pad2) -> Net-(D3:12-Pad2)
- SW3:13 pad 2: Net-(SW3:13-Pad2) -> Net-(D3:13-Pad2)
- SW3:8 pad 2: Net-(SW3:8-Pad2) -> Net-(D3:8-Pad2)
- SW3:9 pad 2: Net-(SW3:9-Pad2) -> Net-(D3:9-Pad2)
- SW4:10 pad 2: Net-(SW4:10-Pad2) -> Net-(D4:10-Pad2)
- SW4:11 pad 2: Net-(SW4:11-Pad2) -> Net-(D4:11-Pad2)
- SW4:12 pad 2: Net-(SW4:12-Pad2) -> Net-(D4:12-Pad2)
- SW4:13 pad 2: Net-(SW4:13-Pad2) -> Net-(D4:13-Pad2)
- SW4:7 pad 2: Net-(SW4:7-Pad2) -> Net-(D4:7-Pad2)
- SW4:8 pad 2: Net-(SW4:8-Pad2) -> Net-(D4:8-Pad2)
- SW4:9 pad 2: Net-(SW4:9-Pad2) -> Net-(D4:9-Pad2)
- SW5:10 pad 2: Net-(SW5:10-Pad2) -> Net-(D5:10-Pad2)
- SW5:11 pad 2: Net-(SW5:11-Pad2) -> Net-(D5:11-Pad2)
- SW5:12 pad 2: Net-(SW5:12-Pad2) -> Net-(D5:12-Pad2)
- SW5:13 pad 2: Net-(SW5:13-Pad2) -> Net-(D5:13-Pad2)
- SW5:7 pad 2: Net-(SW5:7-Pad2) -> Net-(D5:7-Pad2)
- SW5:8 pad 2: Net-(SW5:8-Pad2) -> Net-(D5:8-Pad2)
- SW5:9 pad 2: Net-(SW5:9-Pad2) -> Net-(D5:9-Pad2)
- U1 pad 10: /COL6 -> /COL4
- U1 pad 11: /COL5 -> /COL10
- U1 pad 12: /COL4 -> (no net)
- U1 pad 13: /COL10 -> /RST
- U1 pad 15: /LED_A -> GND
- U1 pad 16: /LED_B -> (no net)
- U1 pad 17: /LED_C -> (no net)
- U1 pad 18: (no net) -> /SCL
- U1 pad 19: (no net) -> /SDA
- U1 pad 2: (no net) -> VCC
- U1 pad 20: (no net) -> /COL11
- U1 pad 21: VCC -> /COL1
- U1 pad 22: GND -> (no net)
- U1 pad 23: Net-(C1-Pad2) -> GND
- U1 pad 24: Net-(C2-Pad1) -> VCC
- U1 pad 25: /SCLM -> (no net)
- U1 pad 26: /SDAM -> Net-(R9-Pad2)
- U1 pad 27: /COL11 -> (no net)
- U1 pad 28: /COL1 -> Net-(R10-Pad2)
- U1 pad 29: (no net) -> /LED_A
- U1 pad 3: VCC -> /D-
- U1 pad 30: (no net) -> /LED_B
- U1 pad 31: GND -> /COL0
- U1 pad 33: (no net) -> Net-(R8-Pad1)
- U1 pad 34: (no net) -> VCC
- U1 pad 35: (no net) -> GND
- U1 pad 36: (no net) -> /ROW0
- U1 pad 37: (no net) -> /ROW1
- U1 pad 38: (no net) -> /ROW2
- U1 pad 39: (no net) -> /ROW3
- U1 pad 4: /D- -> /D+
- U1 pad 40: (no net) -> /ROW4
- U1 pad 41: /COL0 -> /ROW5
- U1 pad 42: (no net) -> VCC
- U1 pad 43: Net-(R8-Pad1) -> GND
- U1 pad 44: (no net) -> VCC
- U1 pad 45: (no net) -> GND
- U1 pad 5: /D+ -> GND
- U1 pad 6: GND -> (no net)
- U1 pad 7: Net-(C3-Pad1) -> VCC
- U1 pad 8: VCC -> /COL6
- U1 pad 9: (no net) -> /COL5
- U2 pad 12: /SCLM -> /SCL
- U2 pad 13: /SDAM -> /SDA
Routing:
- net /COL1: track 321.6 -> 0.00 mm
- net /COL11: track 319.0 -> 0.00 mm
- net /COL4: track 292.1 -> 0.00 mm, vias 2 -> 0
- net /COL6: track 269.3 -> 0.00 mm, vias 2 -> 0
- net /COL10: track 249.0 -> 0.00 mm, vias 2 -> 0
- net /COL5: track 248.3 -> 0.00 mm, vias 2 -> 0
- net /COL0: track 196.3 -> 0.00 mm
- net /ROW1: track 307.8 -> 156.2 mm, vias 2 -> 0
- net VCC: track 148.3 -> 0.00 mm, vias 12 -> 0
- net Net-(LED_B1-Pad2): track 141.7 -> 0.00 mm, vias 2 -> 0
- net /ROW3: track 232.0 -> 91.5 mm, vias 2 -> 0
- net /SDAM: track 136.1 -> 0.00 mm, vias 2 -> 0
- net /ROW4: track 255.1 -> 121.7 mm, vias 2 -> 0
- net Net-(LED_C1-Pad2): track 131.7 -> 0.00 mm
- net /ROW0: track 394.6 -> 269.4 mm, vias 2 -> 1
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Other:
- board text removed: "Components are intended to be placed on the side they are drawn. It is however possible to invert the design. See the webpage for further instructions. www.ergodox.io"
- board text removed: "Design by Dominic Beauchamp, based on the Key64 by Nestor A. Diaz"
- board text removed: "Drawn in KiCAD by Fredrik Atmer, Bathroom Epiphanies"
- board text removed: "Revision 01-05-2017 ProfetKeyboards"
