File: ErgoDOX pcb/ErgoDOX.sch (KiCad schematic (older format))
At the start: 64 parts, among them J1 USB, J2 3.5mm, J3 JMP, J4 JMP, SW0:10 SW0:3, SW0:11 SW0:2, SW0:12 SW0:1, SW0:7 SW0:6, SW0:8 SW0:5, SW0:9 SW0:4, SW1:10 SW1:3, SW1:11 SW1:2, SW1:12 SW1:1, SW1:13 SW1:0, SW1:9 SW1:4, SW2:10 SW2:3, SW2:11 SW2:2, SW2:12 SW2:1, SW2:13 SW2:0, SW2:7 SW2:6, SW2:8 SW2:5, SW2:9 SW2:4, SW3:10 SW3:3, SW3:11 SW3:2, SW3:12 SW3:1, SW3:13 SW3:0, SW3:8 SW3:5, SW3:9 SW3:4, SW4:10 SW4:3, SW4:11 SW4:2, SW4:12 SW4:1, SW4:13 SW4:0, SW4:7 SW4:6, SW4:8 SW4:5, SW4:9 SW4:4, SW5:10 SW5:3, SW5:11 SW5:2, SW5:12 SW5:1, SW5:13 SW5:0, SW5:7 SW5:6, SW5:8 SW5:5, SW5:9 SW5:4, U1 TEENSY2.0, U2 MCP23018

Commit message: Replaced teensy with atmega
Imported project into new version of KiCad
Initial routing of traces is done
Switch footprints need some investigation - overlap is throwing design rule errors
Parts:
- removed H99: MECHANICAL, symbol ANYTHING
- removed J1: USB, symbol 6PIN
- removed J2: 3.5mm, symbol 6PIN
- removed J3, J4: JMP, symbol 3PIN
- removed JP1, JP2: JUMPER, symbol JUMPER
- removed S1, S2: STAB200, symbol ANYTHING
- removed U1: TEENSY2.0, symbol TEENSY2.0
- added C1, C2: 10p, Capacitors_SMD:C_0603, symbol Device:C_Small
- added C3, C4: 1u, Capacitors_SMD:C_0603, symbol Device:C_Small
- added C5, C6: 100n, Capacitors_SMD:C_0603, symbol Device:C_Small
- added J1: AudioJack4, ErgoDOX pcb:ASJ-112-M, symbol Connector:AudioJack4
- added J5: USB_B_Micro, Connectors:USB_Micro-B, symbol Connector:USB_B_Micro
- added R3, R4: 22, Resistors_SMD:R_0603, symbol Device:R
- added R5: 1k, Resistors_SMD:R_0603, symbol Device:R
- added U1: AT90USB1286-MU, Housings_DFN_QFN:QFN-64-1EP_9x9mm_Pitch0.5mm, symbol MCU_Microchip_AVR:AT90USB1286-MU
- added Y1: 16MHz, Crystals:Crystal_SMD_2012-2pin_2.0x1.2mm, symbol Device:Crystal_Small
- D1:7, D1:8: footprint (none) -> Diodes_SMD:D_0603; symbol DIODE -> component:DIODE
- LED_A1, LED_B1, LED_C1: footprint (none) -> LEDs:LED_0603; symbol LED -> component:LED
- R1, R2, RA1, RB1, RC1: footprint (none) -> Resistors_SMD:R_0603; symbol RESISTOR -> component:RESISTOR
- SW0:10, SW0:11, SW0:12, SW0:7, SW0:8, SW0:9, SW1:10, SW1:11, SW1:12, SW1:13, SW1:9, SW2:10, SW2:11, SW2:12, SW2:13, SW2:7, SW2:8, SW2:9, SW3:10, SW3:11, SW3:12, SW3:13, SW3:8, SW3:9, SW4:10, SW4:11, SW4:12, SW4:13, SW4:7, SW4:8, SW4:9, SW5:10, SW5:11, SW5:12, SW5:13, SW5:7, SW5:8, SW5:9: footprint (none) -> ErgoDOX pcb:MX_FLIP_DIODE; symbol SWITCH_DIODE -> component:SWITCH_DIODE
- SW_RST1: symbol SWITCH_PUSH -> component:SWITCH_PUSH
- SX0:10, SX0:11, SX1:7, SX1:8: footprint (none) -> ErgoDOX pcb:MX_FLIP_DIODE; symbol SWITCH_PUSH -> component:SWITCH_PUSH
- U2: footprint (none) -> Housings_SOIC:SOIC-28W_7.5x17.9mm_Pitch1.27mm; symbol MCP23018 -> component:MCP23018
Connections:
- net labels added: AREF, D+, D-, d+, d-
- wire segments 172 -> 270
- no-connect marks 15 -> 33

Commit message: migrated to newer KiCAD
Parts:
- removed R1, R2: 2.2kΩ, Resistors_SMD:R_0603, symbol component:RESISTOR
- removed R3, R4: 22, Resistors_SMD:R_0603, symbol Device:R
- removed R5: 1k, Resistors_SMD:R_0603, symbol Device:R
- removed SW_RST1: SWITCH_PUSH, Buttons_Switches_SMD:SW_SPST_B3U-1000P, symbol component:SWITCH_PUSH
- removed U2: MCP23018, Housings_SOIC:SOIC-28W_7.5x17.9mm_Pitch1.27mm, symbol component:MCP23018
- added R1, R2: 22, Resistors_SMD:R_0603, symbol Device:R_US
- added R6, R7, R8: 1k, Resistors_SMD:R_0603, symbol Device:R_US
- added SW1: SW_Push, symbol Switch:SW_Push
- added U2: MCP23018, Housings_SSOP:SSOP-24_5.3x8.2mm_Pitch0.65mm, symbol ErgoDOX:MCP23018
- D1:7, D1:8: symbol component:DIODE -> Device:D
- LED_A1: value LEDa -> LED; symbol component:LED -> Device:LED
- LED_B1: value LEDb -> LED; symbol component:LED -> Device:LED
- LED_C1: value LEDc -> LED; symbol component:LED -> Device:LED
- R3: renamed from RA1; value LEDa -> 1k; symbol component:RESISTOR -> Device:R_US
- R4: renamed from RB1; value LEDb -> 1k; symbol component:RESISTOR -> Device:R_US
- R5: renamed from RC1; value LEDc -> 1k; symbol component:RESISTOR -> Device:R_US
- SW0:10, SW0:11, SW0:12, SW0:7, SW0:8, SW0:9, SW1:10, SW1:11, SW1:12, SW1:13, SW1:9, SW2:10, SW2:11, SW2:12, SW2:13, SW2:7, SW2:8, SW2:9, SW3:10, SW3:11, SW3:12, SW3:13, SW3:8, SW3:9, SW4:10, SW4:11, SW4:12, SW4:13, SW4:7, SW4:8, SW4:9, SW5:10, SW5:11, SW5:12, SW5:13, SW5:7, SW5:8, SW5:9: symbol component:SWITCH_DIODE -> ErgoDOX:SWITCH_DIODE
- SX0:10, SX0:11, SX1:7, SX1:8: symbol component:SWITCH_PUSH -> ErgoDOX:SWITCH_PUSH
Connections:
- net COL0: now also U2.20 (GPA0); no longer SW1:13.4 (K), SW2:13.4 (K), SW3:13.4 (K), SW4:13.4 (K)
- net COL1: now also U2.21 (GPA1); no longer SW0:12.4 (K), SW1:12.4 (K), SW2:12.4 (K), SW3:12.4 (K), SW4:12.4 (K)
- net COL10: now also U2.23 (GPA3); no longer SW0:10.4 (K), SW1:10.4 (K), SW2:10.4 (K), SW3:10.4 (K), SW4:10.4 (K)
- net COL11: now also U2.22 (GPA2); no longer SW0:11.4 (K), SW1:11.4 (K), SW2:11.4 (K), SW3:11.4 (K), SW4:11.4 (K)
- net COL4: now also U2.24 (GPA4); no longer SW0:9.4 (K), SW1:9.4 (K), SW2:9.4 (K), SW3:9.4 (K), SW4:9.4 (K)
- net COL5: now also D1:8.1 (K), U2.25 (GPA5); no longer D1:8.2 (K), SW0:8.4 (K), SW2:8.4 (K), SW3:8.4 (K), SW4:8.4 (K)
- net COL6: now also D1:7.1 (K), U2.26 (GPA6); no longer D1:7.2 (K), SW0:7.4 (K), SW2:7.4 (K), SW4:7.4 (K)
- net D+: now also R1.1
- net D-: now also R2.1
- net GND: now also LED_A1.1 (K), LED_B1.1 (K), LED_C1.1 (K), R8.2, SW1.2, U2.1 (GND), U2.15 (ADDR); no longer C4.2, C5.2, C6.2, LED_A1.2 (K), LED_B1.2 (K), LED_C1.2 (K), SX0:10.0 (GND), SX0:11.0 (GND), SX1:7.0 (GND), SX1:8.0 (GND)
- net LED_A: now also U2.10 (GPB7)
- net LED_B: now also U2.9 (GPB6)
- net ROW0: now also U2.8 (GPB5); no longer SX0:10.1, SX0:11.1
- net ROW1: now also U2.7 (GPB4)
- net ROW2: now also U2.6 (GPB3)
- net ROW3: now also U2.5 (GPB2)
- net ROW4: now also U2.4 (GPB1)
- net ROW5: now also U2.3 (GPB0)
- net RST: now also SW1.1
- net SCLM: now also R7.2, U2.12 (SCL)
- net SDAM: now also R6.1, U2.13 (SDA)
- net VCC: now also R6.2, R7.1, U2.11 (VCC), U2.16 (RESET)
- net d+: now also R1.2
- net d-: now also R2.2
- net at SW0:10.3 (A), SX0:10.2: no longer SW0:10.2
- net at SW0:11.3 (A), SX0:11.2: no longer SW0:11.2
- net at R3.2: now also LED_A1.2 (A); no longer LED_A1.1 (A)
- net at R4.2: now also LED_B1.2 (A); no longer LED_B1.1 (A)
- net at R5.2: now also LED_C1.2 (A); no longer LED_C1.1 (A)
- net at SX1:8.2: now also D1:8.2 (A); no longer D1:8.1 (A)
- net at SX1:7.2: now also D1:7.2 (A); no longer D1:7.1 (A)
- net at U1.43 (PE2/~HWB): now also R8.1
- new net: C4.2, C5.2, C6.2
Other:
- moved on the sheet: D1:7, D1:8

Commit message: Changed footprints for easier manufacturability
* Diodes are now surface-mount. Don't buy the switches with built-in diodes.
* Changed processor from at90usb1286 to atmega32u4 (due to availability and cost)
* Renamed footprint library
Parts:
- removed SX0:10: SX0:3, ErgoDOX pcb:MX_FLIP_DIODE, symbol ErgoDOX:SWITCH_PUSH
- removed SX0:11: SX0:2, ErgoDOX pcb:MX_FLIP_DIODE, symbol ErgoDOX:SWITCH_PUSH
- removed U1: AT90USB1286-MU, Housings_DFN_QFN:QFN-64-1EP_9x9mm_Pitch0.5mm, symbol MCU_Microchip_AVR:AT90USB1286-MU
- added D0:10, D0:11, D0:12, D0:7, D0:8, D0:9, D1:10, D1:11, D1:12, D1:13, D1:9, D2:10, D2:11, D2:12, D2:13, D2:7, D2:8, D2:9, D3:10, D3:11, D3:12, D3:13, D3:8, D3:9, D4:10, D4:11, D4:12, D4:13, D4:7, D4:8, D4:9, D5:10, D5:11, D5:12, D5:13, D5:7, D5:8, D5:9: D, Diodes_SMD:D_SOD-123, symbol Device:D
- added R10, R9: 0, Resistors_SMD:R_0603, symbol Device:R_US
- added U?: ATmega32U4-MU, Package_DFN_QFN:QFN-44-1EP_7x7mm_P0.5mm_EP5.2x5.2mm, symbol MCU_Microchip_ATmega:ATmega32U4-MU
- D1:7, D1:8: footprint Diodes_SMD:D_0603 -> Diodes_SMD:D_SOD-123
- SW0:10, SW0:11, SW0:12, SW0:7, SW0:8, SW0:9, SW1:10, SW1:11, SW1:12, SW1:13, SW1:9, SW2:10, SW2:11, SW2:12, SW2:13, SW2:7, SW2:8, SW2:9, SW3:10, SW3:11, SW3:12, SW3:13, SW3:8, SW3:9, SW4:10, SW4:11, SW4:12, SW4:13, SW4:7, SW4:8, SW4:9, SW5:10, SW5:11, SW5:12, SW5:13, SW5:7, SW5:8, SW5:9: footprint ErgoDOX pcb:MX_FLIP_DIODE -> ErgoDOX:MX_FLIP_XX; symbol ErgoDOX:SWITCH_DIODE -> ErgoDOX:SWITCH_PUSH
- SX1:7, SX1:8: footprint ErgoDOX pcb:MX_FLIP_DIODE -> ErgoDOX:MX_FLIP_XX
- Y1: footprint Crystals:Crystal_SMD_2012-2pin_2.0x1.2mm -> Crystals:Crystal_SMD_3225-4pin_3.2x2.5mm
Connections:
- net COL0: now also D1:13.1 (K), D2:13.1 (K), D3:13.1 (K), D4:13.1 (K), D5:13.1 (K), U?.31 (PC6); no longer SW5:13.4 (K)
- net COL1: now also D0:12.1 (K), D1:12.1 (K), D2:12.1 (K), D3:12.1 (K), D4:12.1 (K), D5:12.1 (K), U?.21 (PD3); no longer SW5:12.4 (K)
- net COL10: now also D0:10.1 (K), D1:10.1 (K), D2:10.1 (K), D3:10.1 (K), D4:10.1 (K), D5:10.1 (K), U?.11 (PB3); no longer SW5:10.4 (K)
- net COL11: now also D0:11.1 (K), D1:11.1 (K), D2:11.1 (K), D3:11.1 (K), D4:11.1 (K), D5:11.1 (K), U?.20 (PD2); no longer SW5:11.4 (K)
- net COL4: now also D0:9.1 (K), D1:9.1 (K), D2:9.1 (K), D3:9.1 (K), D4:9.1 (K), D5:9.1 (K), U?.10 (PB2); no longer SW5:9.4 (K)
- net COL5: now also D0:8.1 (K), D2:8.1 (K), D3:8.1 (K), D4:8.1 (K), D5:8.1 (K), U?.9 (PB1); no longer SW5:8.4 (K)
- net COL6: now also D0:7.1 (K), D2:7.1 (K), D4:7.1 (K), D5:7.1 (K), U?.8 (PB0); no longer SW5:7.4 (K)
- net D+: now also U?.4 (D+)
- net D-: now also U?.3 (D-)
- net GND: now also C4.2, C5.2, C6.2, R9.1, U?.15 (GND), U?.23 (GND), U?.35 (GND), U?.43 (GND), U?.45 (GND), U?.5 (UGND); no longer SW0:10.0 (GND), SW0:11.0 (GND), SW0:12.0 (GND), SW0:7.0 (GND), SW0:8.0 (GND), SW0:9.0 (GND), SW1:10.0 (GND), SW1:11.0 (GND), SW1:12.0 (GND), SW1:13.0 (GND), SW1:9.0 (GND), SW2:10.0 (GND), SW2:11.0 (GND), SW2:12.0 (GND), SW2:13.0 (GND), SW2:7.0 (GND), SW2:8.0 (GND), SW2:9.0 (GND), SW3:10.0 (GND), SW3:11.0 (GND), SW3:12.0 (GND), SW3:13.0 (GND), SW3:8.0 (GND), SW3:9.0 (GND), SW4:10.0 (GND), SW4:11.0 (GND), SW4:12.0 (GND), SW4:13.0 (GND), SW4:7.0 (GND), SW4:8.0 (GND), SW4:9.0 (GND), SW5:10.0 (GND), SW5:11.0 (GND), SW5:12.0 (GND), SW5:13.0 (GND), SW5:7.0 (GND), SW5:8.0 (GND), SW5:9.0 (GND)
- net LED_A: now also U?.29 (PB5)
- net LED_B: now also U?.30 (PB6)
- net LED_C: now also U?.12 (PB7)
- net ROW0: now also U?.36 (PF7)
- net ROW1: now also U?.37 (PF6)
- net ROW2: now also U?.38 (PF5)
- net ROW3: now also U?.39 (PF4)
- net ROW4: now also U?.40 (PF1)
- net ROW5: now also U?.41 (PF0)
- net RST: now also U?.13 (~RESET)
- net VCC: now also R10.1, U?.14 (VCC), U?.2 (UVCC), U?.24 (AVCC), U?.34 (VCC), U?.42 (AREF), U?.44 (AVCC), U?.7 (VBUS)
- net at SW0:10.2: now also D0:10.2 (A)
- net at SW4:7.2: now also D4:7.2 (A); no longer SW4:7.3 (A)
- net at SW4:8.2: now also D4:8.2 (A); no longer SW4:8.3 (A)
- net at SW4:12.2: now also D4:12.2 (A); no longer SW4:12.3 (A)
- net at SW4:11.2: now also D4:11.2 (A); no longer SW4:11.3 (A)
- net at SW4:10.2: now also D4:10.2 (A); no longer SW4:10.3 (A)
- net at SW4:9.2: now also D4:9.2 (A); no longer SW4:9.3 (A)
- net at SW4:13.2: now also D4:13.2 (A); no longer SW4:13.3 (A)
- net at SW3:12.2: now also D3:12.2 (A); no longer SW3:12.3 (A)
- net at SW3:11.2: now also D3:11.2 (A); no longer SW3:11.3 (A)
- net at SW3:10.2: now also D3:10.2 (A); no longer SW3:10.3 (A)
- net at SW3:9.2: now also D3:9.2 (A); no longer SW3:9.3 (A)
- net at SW3:8.2: now also D3:8.2 (A); no longer SW3:8.3 (A)
- net at SW1:9.2: now also D1:9.2 (A); no longer SW1:9.3 (A)
- net at SW1:10.2: now also D1:10.2 (A); no longer SW1:10.3 (A)
- net at SW1:12.2: now also D1:12.2 (A); no longer SW1:12.3 (A)
- net at SW2:12.2: now also D2:12.2 (A); no longer SW2:12.3 (A)
- net at SW2:11.2: now also D2:11.2 (A); no longer SW2:11.3 (A)
- net at SW2:10.2: now also D2:10.2 (A); no longer SW2:10.3 (A)
- net at SW2:9.2: now also D2:9.2 (A); no longer SW2:9.3 (A)
- net at SW2:8.2: now also D2:8.2 (A); no longer SW2:8.3 (A)
- net at SW2:7.2: now also D2:7.2 (A); no longer SW2:7.3 (A)
- net at SW3:13.2: now also D3:13.2 (A); no longer SW3:13.3 (A)
- net at SW1:13.2: now also D1:13.2 (A); no longer SW1:13.3 (A)
- net at SW2:13.2: now also D2:13.2 (A); no longer SW2:13.3 (A)
- net at SW0:11.2: now also D0:11.2 (A)
- net at SW0:12.2: now also D0:12.2 (A); no longer SW0:12.3 (A)
- net at SW0:7.2: now also D0:7.2 (A); no longer SW0:7.3 (A)
- net at SW0:8.2: now also D0:8.2 (A); no longer SW0:8.3 (A)
- net at SW0:9.2: now also D0:9.2 (A); no longer SW0:9.3 (A)
- net at SW1:11.2: now also D1:11.2 (A); no longer SW1:11.3 (A)
- net at SW5:13.2: now also D5:13.2 (A); no longer SW5:13.3 (A)
- net at SW5:9.2: now also D5:9.2 (A); no longer SW5:9.3 (A)
- net at SW5:10.2: now also D5:10.2 (A); no longer SW5:10.3 (A)
- net at SW5:11.2: now also D5:11.2 (A); no longer SW5:11.3 (A)
- net at SW5:12.2: now also D5:12.2 (A); no longer SW5:12.3 (A)
- net at SW5:8.2: now also D5:8.2 (A); no longer SW5:8.3 (A)
- net at SW5:7.2: now also D5:7.2 (A); no longer SW5:7.3 (A)
- net at C1.2, Y1.2: now also U?.16 (XTAL2)
- net at C2.1, Y1.1: now also U?.17 (XTAL1)
- net at R8.1: now also U?.33 (~HWB~/PE2)
- net at C3.1: now also U?.6 (UCAP)
- net SCLM renamed SCL
- net SCL: now also U?.18 (PD0)
- net SDAM renamed SDA
- net SDA: now also U?.19 (PD1)
- net d+ renamed USB+
- net d- renamed USB-
- new net: R10.2, U?.28 (PB4)
- new net: R9.2, U?.26 (PD6)
- no-connect marks 33 -> 12
Other:
- moved on the sheet: C1, C2, C3, C4, C5, C6, D1:7, D1:8, J1, J5, LED_A1, LED_B1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

Commit message: Placed diodes, started routing
Parts:
- removed J5: USB_B_Micro, Connectors:USB_Micro-B, symbol Connector:USB_B_Micro
- added J2: USB_B_Micro, Connectors_USB:USB_Micro-B_Wuerth-629105150521, symbol Connector:USB_B_Micro
- J1: footprint ErgoDOX pcb:ASJ-112-M -> ErgoDOX:54-00174
- SW0:10, SW0:11, SW0:12, SW0:7, SW0:8, SW0:9, SW1:10, SW1:11, SW1:12, SW1:13, SW1:9, SW2:10, SW2:11, SW2:12, SW2:13, SW2:7, SW2:8, SW2:9, SW3:10, SW3:11, SW3:12, SW3:13, SW3:8, SW3:9, SW4:10, SW4:11, SW4:12, SW4:13, SW4:7, SW4:8, SW4:9, SW5:10, SW5:11, SW5:12, SW5:13, SW5:7, SW5:8, SW5:9, SX1:7, SX1:8: footprint ErgoDOX:MX_FLIP_XX -> ErgoDOX:MX_TOP
- SW1: value SW_Push -> TS-1187A-B-A-B; footprint (none) -> Buttons_Switches_THT:SW_PUSH_6mm
- U1: renamed from U?; footprint Package_DFN_QFN:QFN-44-1EP_7x7mm_P0.5mm_EP5.2x5.2mm -> Housings_DFN_QFN:QFN-44-1EP_7x7mm_Pitch0.5mm
Connections:
- net GND: now also J2.5 (GND), J2.6 (Shield)
- net USB+: now also J2.3 (D+)
- net USB-: now also J2.2 (D-)
- net VCC: now also J2.1 (VBUS)
